File: hardware/boosterpack/Switch Boosterpack.brd (EAGLE design)
At the start: 49.5 x 49.5 mm, 36 parts, among them IC1 LAUNCHPAD-50MM, Q1 IRFR3709, Q2 IRFR3709, Q3 IRFR3709, Q4 IRFR3709

Commit message: BS0 is now tied to GND, C1, C2 are 1 uF and R7 is 390k.
Those are main v1.0 errors. They must be fixed otherwise v1.0 boards are not working.
Parts:
- C1, C2: value 100nF -> 1 uF
- R7: value 10k -> 390k
Connections:
- net GND: now also IC3.10
Changed lines of the file:
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@@
 <attribute name="VALUE" x="3.23" y="39.73" size="0.4064" layer="27" rot="R90"/>
 </element>
-<element name="C1" library="rcl" package="C0603" value="100nF" x="4.826" y="29.972" smashed="yes" rot="MR90">
+<element name="C1" library="rcl" package="C0603" value="1 uF" x="4.826" y="29.972" smashed="yes" rot="MR90">
 <attribute name="NAME" x="4.699" y="31.877" size="0.8128" layer="26" rot="MR90"/>
 <attribute name="VALUE" x="2.921" y="29.337" size="1.27" layer="28" rot="MR90"/>
 </element>
-<element name="C2" library="rcl" package="C0603" value="100nF" x="7.366" y="29.972" smashed="yes" rot="MR90">
+<element name="C2" library="rcl" package="C0603" value="1 uF" x="7.366" y="29.972" smashed="yes" rot="MR90">
 <attribute name="NAME" x="6.985" y="31.877" size="0.8128" layer="26" rot="MR90"/>
 <attribute name="VALUE" x="5.461" y="29.337" size="1.27" layer="28" rot="MR90"/>
@@
 <attribute name="VALUE" x="26.543" y="26.797" size="1.27" layer="28" rot="MR180"/>
 </element>
-<element name="R7" library="rcl" package="R0603" value="10k" x="21.844" y="29.972" smashed="yes" rot="MR270">
+<element name="R7" library="rcl" package="R0603" value="390k" x="21.844" y="29.972" smashed="yes" rot="MR270">
 <attribute name="NAME" x="21.463" y="31.877" size="0.8128" layer="26" rot="MR90"/>
 <attribute name="VALUE" x="23.749" y="30.607" size="1.27" layer="28" rot="MR270"/>
@@
 <vertex x="49.53" y="0"/>
 </polygon>
+<contactref element="IC3" pad="10"/>
 </signal>
 <signal name="N$1">
@@
 <contactref element="R9" pad="2"/>
 <contactref element="R11" pad="2"/>
-<contactref element="C5" pad="1"/>
-<contactref element="C6" pad="1"/>
-<wire x1="11.493" y1="26.398" x2="11.493" y2="29.059" width="0.3048" layer="16"/>
-<wire x1="11.493" y1="29.059" x2="11.43" y2="29.122" width="0.3048" layer="16"/>
-<wire x1="7.993" y1="26.398" x2="7.993" y2="27.717" width="0.3048" layer="16"/>
-<wire x1="7.993" y1="27.717" x2="9.398" y2="29.122" width="0.3048" layer="16"/>
 <wire x1="13.97" y1="1.905" x2="13.97" y2="5.08" width="0.8128" layer="1"/>
 <wire x1="13.97" y1="5.08" x2="12.192" y2="6.858" width="0.8128" layer="1"/>
@@
 <wire x1="5.842" y1="7.874" x2="5.842" y2="14.224" width="0.8128" layer="1"/>
 <wire x1="4.064" y1="31.242" x2="5.588" y2="32.766" width="0.8128" layer="1"/>
-<wire x1="5.588" y1="32.766" x2="10.414" y2="32.766" width="0.8128" layer="1"/>
+<wire x1="5.588" y1="32.766" x2="8.382" y2="32.766" width="0.8128" layer="1"/>
+<wire x1="8.382" y1="32.766" x2="10.414" y2="32.766" width="0.8128" layer="1"/>
 <wire x1="10.414" y1="32.766" x2="12.446" y2="32.766" width="0.8128" layer="1"/>
 <wire x1="12.446" y1="32.766" x2="15.748" y2="32.766" width="0.8128" layer="1"/>
@@
 <wire x1="4.953" y1="7.493" x2="6.35" y2="7.493" width="0.4064" layer="1"/>
 <wire x1="6.35" y1="7.493" x2="6.731" y2="6.985" width="0.4064" layer="1"/>
-<wire x1="10.093" y1="26.398" x2="10.093" y2="27.619" width="0.3048" layer="16"/>
-<wire x1="10.093" y1="27.619" x2="10.414" y2="27.94" width="0.3048" layer="16"/>
-<via x="10.414" y="27.94" extent="1-16" drill="0.5"/>
-<wire x1="10.414" y1="27.94" x2="10.414" y2="32.766" width="0.4064" layer="1"/>
-<wire x1="11.43" y1="29.122" x2="12.358" y2="29.122" width="0.3048" layer="16"/>
-<wire x1="12.358" y1="29.122" x2="12.446" y2="29.21" width="0.3048" layer="16"/>
 <via x="12.446" y="29.21" extent="1-16" drill="0.5"/>
 <wire x1="12.446" y1="29.21" x2="12.446" y2="32.766" width="0.4064" layer="1"/>
-<wire x1="9.398" y1="29.122" x2="9.486" y2="29.122" width="0.3048" layer="16"/>
-<wire x1="10.414" y1="27.94" x2="10.414" y2="28.106" width="0.3048" layer="16"/>
-<wire x1="10.414" y1="28.106" x2="9.398" y2="29.122" width="0.3048" layer="16"/>
 <wire x1="4.064" y1="31.242" x2="1.524" y2="28.702" width="0.8128" layer="1"/>
 <wire x1="1.524" y1="28.702" x2="1.524" y2="16.637" width="0.8128" layer="1"/>
@@
 <wire x1="5.842" y1="14.224" x2="5.842" y2="14.986" width="0.8128" layer="1"/>
 <wire x1="5.842" y1="14.986" x2="5.588" y2="15.24" width="0.8128" layer="1"/>
+<contactref element="C5" pad="1"/>
+<contactref element="C6" pad="1"/>
+<wire x1="9.398" y1="29.122" x2="9.486" y2="29.122" width="0.3048" layer="16"/>
+<wire x1="11.493" y1="26.398" x2="11.493" y2="27.495" width="0.3048" layer="16"/>
+<wire x1="11.493" y1="27.495" x2="11.938" y2="27.94" width="0.3048" layer="16"/>
+<wire x1="12.446" y1="29.21" x2="12.446" y2="28.448" width="0.3048" layer="16"/>
+<wire x1="12.446" y1="28.448" x2="11.938" y2="27.94" width="0.3048" layer="16"/>
+<wire x1="11.43" y1="29.122" x2="12.358" y2="29.122" width="0.4064" layer="16"/>
+<wire x1="12.358" y1="29.122" x2="12.446" y2="29.21" width="0.4064" layer="16"/>
+<wire x1="9.486" y1="29.122" x2="9.486" y2="28.868" width="0.4064" layer="16"/>
+<wire x1="7.993" y1="26.398" x2="7.993" y2="27.551" width="0.3048" layer="16"/>
+<wire x1="7.993" y1="27.551" x2="8.382" y2="27.94" width="0.3048" layer="16"/>
+<via x="8.382" y="27.94" extent="1-16" drill="0.5"/>
+<wire x1="8.382" y1="27.94" x2="8.382" y2="32.766" width="0.4064" layer="1"/>
+<wire x1="9.486" y1="28.868" x2="9.31" y2="28.868" width="0.3048" layer="16"/>
+<wire x1="9.31" y1="28.868" x2="8.382" y2="27.94" width="0.4064" layer="16"/>
+<wire x1="10.093" y1="26.398" x2="10.093" y2="27.626" width="0.3048" layer="16"/>
+<wire x1="10.093" y1="27.626" x2="9.779" y2="27.94" width="0.3048" layer="16"/>
+<wire x1="9.779" y1="27.94" x2="8.382" y2="27.94" width="0.3048" layer="16"/>
 </signal>
 <signal name="SCL">

Commit message: Fixed schematic, instead of N channel FET there were P channel FET on schematic.
So actually 1.0 board MOSFET side was messed up. Now it is correct. P channel FET was used in "N channel configuration".
Parts:
- Q1, Q2, Q3, Q4: value IRFR3709 -> IRF3709S; device transistor-power:D-PAK_TO252AA -> mosfet:D-PAK_TO252AA
- moved R3 8.73 mm to (39.9, 13.5)
- moved R1 8.48 mm to (39.9, 37.8)
- moved R2 8.48 mm to (39.9, 26.2)
- moved R4 7.77 mm to (39.9, 3.05)
- moved Q4 0.57 mm to (37.3, 7.37)
- moved Q2 0.36 mm to (37.3, 31.0)
- moved Q1 0.25 mm to (37.3, 42.7)
- moved Q3 0.25 mm to (37.3, 18.3)
Connections:
- net GND: now also Q1.3, Q2.3, Q3.3, Q4.3; no longer Q1.4, Q2.4, Q3.4, Q4.4
- net N$1: now also Q1.4; no longer Q1.3
- net N$3: now also Q2.4; no longer Q2.3
- net N$5: now also Q3.4; no longer Q3.3
- net N$7: now also Q4.4; no longer Q4.3
Routing:
- net LOAD1: track 51.9 -> 42.8 mm
- net LOAD4: track 11.7 -> 2.67 mm
- net N$7: track 8.80 -> 17.1 mm
- net LOAD2: track 38.9 -> 31.1 mm
- net N$2: track 1.32 -> 7.69 mm
- net N$4: track 1.58 -> 7.69 mm
- net N$6: track 1.58 -> 7.69 mm
- net N$5: track 9.17 -> 15.2 mm
- net N$3: track 9.35 -> 15.4 mm
- net N$8: track 1.68 -> 7.18 mm
- net N$1: track 10.1 -> 15.2 mm
- net LOAD3: track 24.2 -> 19.9 mm
